Commit message: Updated weight for model and added imu and lidar sensor plugins

File: omnibot_description/urdf/omnibot.xacro (robot description, xacro)
@@ -91,5 +91,5 @@
   </collision>
 </link>
-<link name="lidar_link_1">
+<link name="lidar_frame">
   <inertial>
     <origin xyz="0.01572744785340128 -0.03173001991250517 0.024230508055298527" rpy="0 0 0"/>
@@ -98,5 +98,5 @@
   </inertial>
   <visual>
-    <origin xyz="0.026373 -0.038321 -0.132" rpy="0 0 0"/>
+    <origin xyz="0.0 -0.0 -0.176" rpy="0 0 0"/>
     <geometry>
       <mesh filename="file://$(find omnibot_description)/meshes/lidar_link_1.stl" scale="0.001 0.001 0.001"/>
@@ -105,5 +105,5 @@
   </visual>
   <collision>
-    <origin xyz="0.026373 -0.038321 -0.132" rpy="0 0 0"/>
+    <origin xyz="0.0 -0.0 -0.176" rpy="0 0 0"/>
     <geometry>
       <mesh filename="file://$(find omnibot_description)/meshes/lidar_link_1.stl" scale="0.001 0.001 0.001"/>
@@ -131,4 +131,22 @@
   </collision>
 </link>
+<link name="imu_link">
+  <visual>
+    <origin xyz="0.0 0.0 0.0025" rpy="0.0 0.0 0.0"/>
+    <geometry>
+      <box size="0.01 0.02 0.005"/>
+    </geometry>
+  </visual>
+  <collision>
+    <origin xyz="0.0 0.0 0.0025" rpy="0.0 0.0 0.0"/>
+    <geometry>
+      <box size="0.01 0.01 0.01"/>
+    </geometry>
+  </collision>
+  <inertial>
+    <mass value="0.01"/>
+    <inertia ixx="1e-6" ixy="0" ixz="0" iyy="1e-6" iyz="0" izz="1e-6"/>
+  </inertial>
+</link>
 <joint name="wheel2_base_joint" type="continuous">
   <origin xyz="-0.027709 0.048166 0.0085" rpy="0 0 0"/>
@@ -150,7 +168,7 @@
 </joint>
 <joint name="lidar_base_joint" type="fixed">
-  <origin xyz="-0.026373 0.038321 0.132" rpy="0 0 0"/>
+  <origin xyz="-0.0 0.0 0.176" rpy="0 0 0"/>
   <parent link="base_link"/>
-  <child link="lidar_link_1"/>
+  <child link="lidar_frame"/>
 </joint>
 <joint name="camera_base_joint" type="fixed">
@@ -159,3 +177,8 @@
   <child link="camera_link_1"/>
 </joint>
+<joint name="imu_joint" type="fixed">
+  <parent link="base_link"/>
+  <child link="imu_link"/>
+  <origin xyz="0 0 0.1" rpy="0 0 0"/>
+</joint>
 </robot>

Commit message: yolo node updated Localization and navigation script added

File: omnibot_description/urdf/omnibot.xacro (robot description, xacro)
@@ -34,5 +34,5 @@
   <inertial>
     <origin xyz="-0.008769128668929132 0.015270306522884095 8.274069084416094e-06" rpy="0 0 0"/>
-    <mass value="0.1270196974399702"/>
+    <mass value="0.3"/>
     <inertia ixx="1.6e-05" iyy="1.9e-05" izz="1.5e-05" ixy="-3e-06" iyz="0.0" ixz="-0.0"/>
   </inertial>
@@ -54,5 +54,5 @@
   <inertial>
     <origin xyz="0.01760894584883433 -4.108092348062824e-05 8.274069084419564e-06" rpy="0 0 0"/>
-    <mass value="0.1270196974399702"/>
+    <mass value="0.3"/>
     <inertia ixx="2.1e-05" iyy="1.5e-05" izz="1.5e-05" ixy="-0.0" iyz="-0.0" ixz="0.0"/>
   </inertial>
@@ -74,5 +74,5 @@
   <inertial>
     <origin xyz="-0.008840288621883803 -0.015229966759758365 8.274069084417829e-06" rpy="0 0 0"/>
-    <mass value="0.1270196974399702"/>
+    <mass value="0.3"/>
     <inertia ixx="1.6e-05" iyy="1.9e-05" izz="1.5e-05" ixy="3e-06" iyz="-0.0" ixz="-0.0"/>
   </inertial>
